File: LED-Board.brd (EAGLE design)
At the start: 71 x 34 mm, 30 parts, among them U1 ATSAMD11C14A-SSUT, U3 LDL1117S12R

Commit message: fixed up right angle
Routing:
- net GND: track 13.4 -> 11.6 mm
Changed lines of the file:
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@@
 <wire x1="38.227" y1="40.259" x2="39.0906" y2="40.259" width="0.2032" layer="1"/>
 <wire x1="39.0906" y1="40.259" x2="39.37" y2="40.5384" width="0.2032" layer="1"/>
-<wire x1="39.37" y1="40.5384" x2="42.8752" y2="40.5384" width="0.2032" layer="16"/>
-<wire x1="42.8752" y1="40.5384" x2="46.0248" y2="37.3888" width="0.2032" layer="16"/>
-<wire x1="46.0248" y1="37.3888" x2="43.3832" y2="37.3888" width="0.2032" layer="16"/>
+<wire x1="43.3832" y1="37.3888" x2="47.0408" y2="37.3888" width="0.2032" layer="16"/>
 <wire x1="43.3832" y1="37.3888" x2="43.0784" y2="37.084" width="0.2032" layer="16"/>
 <via x="43.0784" y="37.084" extent="1-16" drill="0.4"/>
 <contactref element="C2" pad="-"/>
+<wire x1="39.37" y1="40.5384" x2="39.624" y2="40.5384" width="0.2032" layer="16"/>
+<wire x1="39.624" y1="40.5384" x2="43.0784" y2="37.084" width="0.2032" layer="16"/>
 </signal>
 <signal name="LED-">
