File: LED-Board.brd (EAGLE design)
At the start: 71 x 34 mm, 30 parts, among them U1 ATSAMD11C14A-SSUT, U3 LDL1117S12R

Commit message: final touches to LED board
Parts:
- removed 1UF2: (no value), microbuilder:0603
- added C6: (no value), microbuilder:0603
- added FD1, FD2, FD3, FD4: FIDUCIAL1X2, SparkFun-Aesthetics:FIDUCIAL-1X2
- moved C1 35.2 mm to (18.8, 27.0)
- moved C2 35.2 mm to (12.0, 27.0)
- moved C4 35.2 mm to (22.0, 2.38)
- moved C5 35.2 mm to (13.8, 11.9)
- moved D1 35.2 mm to (28.0, 14.5)
- moved D2 35.2 mm to (39.6, 12.7)
- moved D3 35.2 mm to (31.7, 12.4)
- moved D6 35.2 mm to (41.6, 8.24)
- moved F1 35.2 mm to (27.9, 23.7)
- moved GND-CLIP 35.2 mm to (50.5, 20.0)
- moved GND-CLIP3 35.2 mm to (50.5, 20.0)
- moved IC4 35.2 mm to (43.0, 10.6)
- moved J1 35.2 mm to (32.8, 1.96)
- moved J2 35.2 mm to (56.5, 4.12)
- moved J3 35.2 mm to (64.1, 6.66)
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Connections:
- net 3.3V: now also C6.1; no longer 1UF2.1
- net GND: now also C6.2; no longer 1UF2.2
Routing:
- net GND: vias 68 -> 72
Other:
- board text removed: "Sense"
