File: angle.brd (EAGLE design)
At the start: 58 x 29.8 mm, 12 parts

Commit message: fixed up right angle
Routing:
- added copper zone on layer 16, net GND1
- added copper zone on layer 16, net PWM1
- added copper zone on layer 16, net VCC-RAW1
- removed copper zone on layer 16, net GND
- removed copper zone on layer 16, net PWM
- removed copper zone on layer 16, net VCC-RAW
Changed lines of the file:
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@@
 <?xml version="1.0" encoding="utf-8"?>
 <!DOCTYPE eagle SYSTEM "eagle.dtd">
-<eagle version="9.2.2">
+<eagle version="9.3.0">
 <drawing>
 <settings>
-<setting alwaysvectorfont="yes"/>
+<setting alwaysvectorfont="no"/>
 <setting keepoldvectorfont="yes"/>
 <setting verticaltext="up"/>
 </settings>
-<grid distance="0.2" unitdist="mm" unit="mm" style="lines" multiple="1" display="yes" altdistance="0.025" altunitdist="inch" altunit="inch"/>
+<grid distance="0.1" unitdist="mm" unit="mm" style="lines" multiple="1" display="yes" altdistance="0.025" altunitdist="inch" altunit="inch"/>
 <layers>
 <layer number="1" name="Top" color="4" fill="1" visible="yes" active="yes"/>
@@
 <layer number="45" name="Holes" color="7" fill="1" visible="yes" active="yes"/>
 <layer number="46" name="Milling" color="3" fill="1" visible="no" active="yes"/>
-<layer number="47" name="Measures" color="7" fill="1" visible="yes" active="yes"/>
+<layer number="47" name="Measures" color="7" fill="1" visible="no" active="yes"/>
 <layer number="48" name="Document" color="7" fill="1" visible="no" active="yes"/>
 <layer number="49" name="Reference" color="7" fill="1" visible="no" active="yes"/>
@@
 <hole x="60" y="78.7" drill="3"/>
 <wire x1="60.5" y1="52.89" x2="64" y2="56.4" width="0" layer="20" curve="90"/>
-<wire x1="64" y1="58.05" x2="64" y2="79.454" width="0" layer="20"/>
+<wire x1="64" y1="58" x2="64" y2="79.454" width="0" layer="20"/>
 <wire x1="64" y1="79.454" x2="61.008" y2="82.7" width="0" layer="20" curve="90"/>
 <wire x1="61.008" y1="82.7" x2="9.5" y2="82.7" width="0" layer="20"/>
@@
 </polygon>
 <dimension x1="64" y1="58.1" x2="35" y2="59" x3="49.5" y3="59.8" textsize="1.778" layer="47" dtype="horizontal"/>
-<wire x1="64" y1="58.05" x2="35" y2="58.05" width="0.001" layer="20"/>
-<wire x1="35" y1="58.05" x2="35" y2="56.4" width="0.001" layer="20"/>
+<wire x1="64" y1="58" x2="35" y2="58" width="0.001" layer="20"/>
+<wire x1="35" y1="58" x2="35" y2="56.4" width="0.001" layer="20"/>
 <wire x1="35" y1="56.4" x2="64" y2="56.4" width="0.001" layer="20"/>
 <text x="16.721" y="70.49" size="1.016" layer="26" rot="MR0">VCC</text>
 <text x="35.033" y="70.54" size="1.016" layer="26" rot="MR0">BUS</text>
 <text x="58.731" y="70.367" size="1.016" layer="26" rot="MR0">GND</text>
+<dimension x1="6" y1="56.39" x2="64" y2="56.4" x3="35.003446875" y3="36.397" textsize="1.778" layer="47"/>
+<dimension x1="6" y1="56.39" x2="27.5" y2="56.4" x3="16.753346875" y3="49.195653125" textsize="1.778" layer="47"/>
+<dimension x1="64" y1="58" x2="42.5" y2="58" x3="53.25" y3="84.7" textsize="1.778" layer="47"/>
+<dimension x1="43.6" y1="81.7" x2="42.5" y2="81.7" x3="43.05" y3="87.9" textsize="1.778" layer="47"/>
+<dimension x1="27.5" y1="81.7" x2="26.4" y2="81.7" x3="26.95" y3="87.6" textsize="1.778" layer="47"/>
 </plain>
 <attributes>
@@
 <contactref element="GND-CLIP3" pad="CLIP-INPUT2"/>
 <contactref element="GND-CLIP3" pad="CLIP-INPUT1"/>
-<polygon width="0.1524" layer="1" thermals="no" rank="4">
-<vertex x="40.08" y="56.873"/>
-<vertex x="40" y="56.873"/>
-<vertex x="40" y="83.2"/>
-<vertex x="67.5" y="83.2"/>
-<vertex x="67.5" y="51.89"/>
-<vertex x="40.08" y="51.89"/>
-</polygon>
 <contactref element="GND-CLIP1" pad="CLIP-INPUT2"/>
 <contactref element="GND-CLIP1" pad="CLIP-INPUT1"/>
 <contactref element="GND-CLIP2" pad="CLIP-INPUT2"/>
 <contactref element="GND-CLIP2" pad="CLIP-INPUT1"/>
-<polygon width="0.7" layer="16" thermals="no">
-<vertex x="40.8" y="86"/>
-<vertex x="71" y="86"/>
-<vertex x="71" y="48"/>
-<vertex x="40.8" y="48"/>
+<polygon width="0.01" layer="1">
+<vertex x="65.4" y="84.1"/>
+<vertex x="43.6" y="84.1"/>
+<vertex x="43.6" y="51"/>
+<vertex x="65.4" y="51"/>
 </polygon>
 </signal>
@@
 <contactref element="PWM-CLIP1" pad="CLIP-INPUT2"/>
 <contactref element="PWM-CLIP1" pad="CLIP-INPUT1"/>
-<polygon width="0.1524" layer="1" thermals="no" rank="3">
-<vertex x="28.127" y="83.2"/>
-<vertex x="28.127" y="51.78"/>
-<vertex x="39.373" y="51.78"/>
-<vertex x="39.373" y="83.2"/>
-</polygon>
 <contactref element="PWM-CLIP2" pad="CLIP-INPUT2"/>
 <contactref element="PWM-CLIP2" pad="CLIP-INPUT1"/>
 <contactref element="PWM-CLIP3" pad="CLIP-INPUT2"/>
 <contactref element="PWM-CLIP3" pad="CLIP-INPUT1"/>
-<polygon width="0.4" layer="16" thermals="no">
-<vertex x="28.8" y="84"/>
-<vertex x="39.2" y="84"/>
-<vertex x="39.2" y="47"/>
-<vertex x="28.8" y="47"/>
+<polygon width="0.01" layer="1">
+<vertex x="42.5" y="83.5"/>
+<vertex x="42.5" y="51.6"/>
+<vertex x="27.5" y="51.5"/>
+<vertex x="27.5" y="83.4"/>
 </polygon>
 </signal>
@@
 <contactref element="VCC-CLIP3" pad="CLIP-INPUT2"/>
 <contactref element="VCC-CLIP3" pad="CLIP-INPUT1"/>
-<polygon width="0.1524" layer="1" thermals="no">
-<vertex x="4.468" y="83.04"/>
-<vertex x="4.468" y="52.08"/>
-<vertex x="27.526" y="52.08"/>
-<vertex x="27.526" y="56.878"/>
-<vertex x="27.518" y="56.878"/>
-<vertex x="27.518" y="83.04"/>
-</polygon>
 <contactref element="VCC-CLIP1" pad="CLIP-INPUT2"/>
 <contactref element="VCC-CLIP1" pad="CLIP-INPUT1"/>
 <contactref element="VCC-CLIP2" pad="CLIP-INPUT2"/>
 <contactref element="VCC-CLIP2" pad="CLIP-INPUT1"/>
-<polygon width="0.4" layer="16" thermals="no">
-<vertex x="3" y="85"/>
-<vertex x="27.4" y="85"/>
-<vertex x="27.4" y="47"/>
-<vertex x="3" y="47"/>
-</polygon>
-</signal>
+<polygon width="0.01" layer="1">
+<vertex x="3.7" y="84.6"/>
+<vertex x="3.7" y="51.6"/>
+<vertex x="26.4" y="51.6"/>
+<vertex x="26.4" y="84.6"/>
+</polygon>
+</signal>
+<signal name="GND1">
+<polygon width="0.01" layer="16">
+<vertex x="4.6" y="84.1"/>
+<vertex x="26.4" y="84.1"/>
+<vertex x="26.4" y="51"/>
+<vertex x="4.6" y="51"/>
+</polygon>
+</signal>
+<signal name="PWM1">
+<polygon width="0.01" layer="16">
+<vertex x="27.5" y="83.5"/>
+<vertex x="27.5" y="51.6"/>
+<vertex x="42.5" y="51.5"/>
+<vertex x="42.5" y="83.4"/>
+</polygon>
+</signal>
+<signal name="VCC-RAW1" class="1">
+<polygon width="0.01" layer="16">
+<vertex x="66.3" y="84.6"/>
+<vertex x="66.3" y="51.6"/>
+<vertex x="43.6" y="51.6"/>
+<vertex x="43.6" y="84.6"/>
+</polygon>
+</signal>
