File: Fan-Module.sch (EAGLE design)
At the start: 14 parts

Commit message: added sdi functionality to fan module
Parts:
- removed C2: 47uF, SparkFun-Capacitors:47UF-POLAR-PANASONIC_D-35V-20%
- removed D2: 3A/40V/500mV, SparkFun-DiscreteSemi:DIODE-SCHOTTKY-B340A
- removed U$2: M20-8900505, MESO:M20-8900505
- added C1: (no value), rcl:C-EUC0603
- added C4, C5: 10uF, rcl:C-EUC0603
- added D3: 3A/40V/500mV, SparkFun-DiscreteSemi:DIODE-SCHOTTKY-B340A
- added F1: (no value), adafruit:PTCFUSE-1812
- added J1: (no value), SparkFun-Connectors:USB_MICRO-B_FEMALE-SMT
- added J10: (no value), SparkFun-Connectors:CONN_02PTH3
- added J2: (no value), SparkFun-Connectors:CONN_05
- added LED1: (no value), led:LEDCHIPLED_0805
- added Q1: (no value), microbuilder:MOSFET-NWIDE
- added R1, R2: 2k, rcl:R-US_R1206
- added R6: 59R, rcl:R-US_R0805
- added U1: ATSAMD11C14A-SSUT_ATSAMD11C14A-SSUT, LED-Board:ATSAMD11C14A-SSUT_ATSAMD11C14A-SSUT
- added U3: LDL1117S12R_LDL1117S12R, LDL1117S12R:LDL1117S12R_LDL1117S12R
Connections:
- removed net 24V: D2.C, U$2.5
- removed net FAN-VCC: C2.+, D1.C, U$2.1
- removed net PWM: D1.A, PWM-CLIP.INPUT, PWM-CLIP1.INPUT
- new net 3.3V: C1.2, C4.2, J2.2, R6.2, U1.VDD, U3.VOUT, U3.VOUT-1
- new net BUS: PWM-CLIP.INPUT, PWM-CLIP1.INPUT, R1.1
- new net FAN: J10.2, Q1.D
- new net N$1: LED1.C, U1.PA04/AIN2
- new net N$2: LED1.A, R6.1
- new net N$3: R1.2, U1.PA15/AIN7
- new net N$4: D3.A, J1.VBUS
- new net N$5: Q1.G, R2.2, U1.PA02/AIN0
- new net N$6: D1.A, F1.1
- new net RESET: J2.5, U1.PA28/!RST
- new net SWCLK: J2.4, U1.PA30/SWCLK
- new net SWDIO: J2.3, U1.PA31/SWDIO
- new net USB+: J1.D+, U1.PA25/USB+
- new net USB-: J1.D-, U1.PA24/USB-
- new net VCC: C5.2, D1.C, D3.C, J10.1, U3.VIN
- net GND: now also C1.1, C4.1, C5.1, J1.GND, J1.SHIELD, J2.1, Q1.S, R2.1, U1.GND, U3.GND; no longer C2.-, U$2.3
- net VCC-RAW: now also F1.2; no longer D2.A
Other:
- moved on the sheet: D1

Commit message: modified c6 to 1uF
Parts:
- C6: value (none) -> 1uF
- renumbered C1 to C6
Changed lines of the file:
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@@
 <part name="LED1" library="led" library_urn="urn:adsk.eagle:library:259" deviceset="LED" device="CHIPLED_0805" package3d_urn="urn:adsk.eagle:package:15821/2"/>
 <part name="U$4" library="microbuilder" deviceset="3.3V" device=""/>
-<part name="C1" library="rcl" library_urn="urn:adsk.eagle:library:334" deviceset="C-EU" device="C0603" package3d_urn="urn:adsk.eagle:package:23616/2"/>
+<part name="C6" library="rcl" library_urn="urn:adsk.eagle:library:334" deviceset="C-EU" device="C0603" package3d_urn="urn:adsk.eagle:package:23616/2" value="1uF"/>
 <part name="GND2" library="SparkFun-Aesthetics" deviceset="GND" device=""/>
 <part name="GND3" library="SparkFun-Aesthetics" deviceset="GND" device=""/>
@@
 <attribute name="VALUE" x="-1.016" y="56.896" size="1.27" layer="96" rot="MR0"/>
 </instance>
-<instance part="C1" gate="G$1" x="-2.54" y="48.26" smashed="yes" rot="R180">
-<attribute name="NAME" x="-4.064" y="47.879" size="1.778" layer="95" rot="R180"/>
-<attribute name="VALUE" x="-4.064" y="52.959" size="1.778" layer="96" rot="R180"/>
+<instance part="C6" gate="G$1" x="-2.54" y="48.26" smashed="yes" rot="R180">
+<attribute name="NAME" x="3.556" y="47.879" size="1.778" layer="95" rot="R180"/>
+<attribute name="VALUE" x="4.826" y="51.689" size="1.778" layer="96" rot="R180"/>
 </instance>
 <instance part="GND2" gate="1" x="-2.54" y="22.86" smashed="yes">
@@
 </segment>
 <segment>
-<pinref part="C1" gate="G$1" pin="1"/>
+<pinref part="C6" gate="G$1" pin="1"/>
 <pinref part="GND3" gate="1" pin="GND"/>
 </segment>
@@
 <segment>
 <pinref part="U$4" gate="G$1" pin="3.3V"/>
-<pinref part="C1" gate="G$1" pin="2"/>
+<pinref part="C6" gate="G$1" pin="2"/>
 <pinref part="U1" gate="G$1" pin="VDD"/>
 <junction x="-2.54" y="53.34"/>
