File: LED-Board.sch (EAGLE design)
At the start: 30 parts, among them U1 ATSAMD11C14A-SSUT, U3 LDL1117S12R

Commit message: final touches to LED board
Parts:
- added FD1, FD2, FD3, FD4: FIDUCIAL1X2, SparkFun-Aesthetics:FIDUCIAL1X2
- renumbered 1UF2 to C6
Changed lines of the file:
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@@
 <part name="FRAME1" library="frames" library_urn="urn:adsk.eagle:library:229" deviceset="A4L-LOC" device=""/>
 <part name="L1" library="microbuilder" deviceset="INDUCTOR" device="TDK_VLC6045"/>
-<part name="1UF2" library="microbuilder" deviceset="CAP_CERAMIC" device="0603"/>
+<part name="C6" library="microbuilder" deviceset="CAP_CERAMIC" device="0603"/>
 <part name="U$1" library="microbuilder" deviceset="GND" device=""/>
 <part name="U$7" library="microbuilder" deviceset="GND" device=""/>
@@
 <part name="F1" library="Adafruit" deviceset="PTCFUSE" device="-1812" value="TLC-MSMD110/24"/>
 <part name="JP1" library="Adafruit" deviceset="PINHD-1X1" device=""/>
+<part name="FD1" library="SparkFun-Aesthetics" deviceset="FIDUCIAL" device="1X2"/>
+<part name="FD2" library="SparkFun-Aesthetics" deviceset="FIDUCIAL" device="1X2"/>
+<part name="FD3" library="SparkFun-Aesthetics" deviceset="FIDUCIAL" device="1X2"/>
+<part name="FD4" library="SparkFun-Aesthetics" deviceset="FIDUCIAL" device="1X2"/>
 </parts>
 <sheets>
@@
 <attribute name="VALUE" x="43.18" y="27.94" size="1.27" layer="96" rot="R90"/>
 </instance>
-<instance part="1UF2" gate="G$1" x="-7.62" y="68.58" smashed="yes">
+<instance part="C6" gate="G$1" x="-7.62" y="68.58" smashed="yes">
 <attribute name="NAME" x="-5.08" y="71.12" size="1.27" layer="95" font="vector"/>
 <attribute name="VALUE" x="-5.08" y="68.58" size="1.27" layer="96" font="vector"/>
@@
 <attribute name="VALUE" x="-59.69" y="55.88" size="1.778" layer="96" rot="R180"/>
 </instance>
+<instance part="FD1" gate="G$1" x="48.26" y="-53.34" smashed="yes"/>
+<instance part="FD2" gate="G$1" x="53.34" y="-53.34" smashed="yes"/>
+<instance part="FD3" gate="G$1" x="58.42" y="-53.34" smashed="yes"/>
+<instance part="FD4" gate="G$1" x="63.5" y="-53.34" smashed="yes"/>
 </instances>
 <busses>
@@
 </segment>
 <segment>
-<pinref part="1UF2" gate="G$1" pin="P$2"/>
+<pinref part="C6" gate="G$1" pin="P$2"/>
 <pinref part="U$1" gate="G$1" pin="GND"/>
 </segment>
@@
 <net name="3.3V" class="1">
 <segment>
-<pinref part="1UF2" gate="G$1" pin="P$1"/>
+<pinref part="C6" gate="G$1" pin="P$1"/>
 <wire x1="-5.08" y1="73.66" x2="-7.62" y2="73.66" width="0.1524" layer="91"/>
 <pinref part="U1" gate="G$1" pin="VDD"/>

Commit message: added values/aligned names and values
Parts:
- C2: value 100uF -> 100uF2
- R6: value (none) -> 59R
Other:
- moved on the sheet: C2

Commit message: exchanged j3 and c1/2 footprint of led module
Parts:
- removed JP1: (no value), Adafruit:PINHD-1X1
- C1: device microbuilder:CAP_ELECTROLYTICPANASONIC_C -> microbuilder:CAP_ELECTROLYTICPANASONIC_D
- C2: value 100uF2 -> 100uF; device microbuilder:CAP_ELECTROLYTICPANASONIC_C -> microbuilder:CAP_ELECTROLYTICPANASONIC_D
- J3: device SparkFun-Connectors:CONN_04 -> SparkFun-Connectors:CONN_05
Connections:
- removed net N$13: JP1.1, U1.PA28/!RST
- new net RESET: J3.5, U1.PA28/!RST
Other:
- moved on the sheet: D3, D6, J1, J2, R6

Commit message: renamed some connectors
Parts:
- J2: device SparkFun-Connectors:CONN_04 -> SparkFun-Connectors:CONN_05
- J3: device SparkFun-Connectors:CONN_05 -> SparkFun-Connectors:CONN_04
Connections:
- net 3.3V: now also J2.2; no longer J3.2
- net GND: now also J2.1; no longer J3.1
- net N$10: now also J3.4; no longer J2.4
- net N$7: now also J3.1; no longer J2.1
- net N$8: now also J3.2; no longer J2.2
- net N$9: now also J3.3; no longer J2.3
- net RESET: now also J2.5; no longer J3.5
- net SWCLK: now also J2.4; no longer J3.4
- net SWDIO: now also J2.3; no longer J3.3
Changed lines of the file:
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@@
 <part name="SUPPLY2" library="SparkFun-Aesthetics" deviceset="VCC" device=""/>
 <part name="D3" library="SparkFun-DiscreteSemi" deviceset="DIODE-SCHOTTKY" device="-B340A" value="3A/40V/500mV"/>
-<part name="J2" library="SparkFun-Connectors" library_urn="urn:adsk.eagle:library:513" deviceset="CONN_04" device="" package3d_urn="urn:adsk.eagle:package:38085/1"/>
+<part name="J3" library="SparkFun-Connectors" library_urn="urn:adsk.eagle:library:513" deviceset="CONN_04" device="" package3d_urn="urn:adsk.eagle:package:38085/1"/>
 <part name="C2" library="microbuilder" deviceset="CAP_ELECTROLYTIC" device="PANASONIC_D" value="100uF"/>
 <part name="F1" library="Adafruit" deviceset="PTCFUSE" device="-1812" value="TLC-MSMD110/24"/>
@@
 <part name="FD3" library="SparkFun-Aesthetics" deviceset="FIDUCIAL" device="1X2"/>
 <part name="FD4" library="SparkFun-Aesthetics" deviceset="FIDUCIAL" device="1X2"/>
-<part name="J3" library="SparkFun-Connectors" deviceset="CONN_05" device=""/>
+<part name="J2" library="SparkFun-Connectors" deviceset="CONN_05" device=""/>
 </parts>
 <sheets>
@@
 <attribute name="NAME" x="-77.9526" y="60.96" size="1.778" layer="95" rot="R90"/>
 </instance>
-<instance part="J2" gate="G$1" x="-66.04" y="63.5" smashed="yes">
+<instance part="J3" gate="G$1" x="-66.04" y="63.5" smashed="yes">
 <attribute name="VALUE" x="-71.12" y="56.134" size="1.778" layer="96" font="vector"/>
 <attribute name="NAME" x="-71.12" y="71.628" size="1.778" layer="95" font="vector"/>
@@
 <instance part="FD3" gate="G$1" x="58.42" y="-53.34" smashed="yes"/>
 <instance part="FD4" gate="G$1" x="63.5" y="-53.34" smashed="yes"/>
-<instance part="J3" gate="G$1" x="-68.58" y="45.72" smashed="yes">
+<instance part="J2" gate="G$1" x="-68.58" y="45.72" smashed="yes">
 <attribute name="VALUE" x="-71.12" y="35.814" size="1.778" layer="96" font="vector"/>
 <attribute name="NAME" x="-71.12" y="53.848" size="1.778" layer="95" font="vector"/>
@@
 </segment>
 <segment>
-<pinref part="J3" gate="G$1" pin="1"/>
+<pinref part="J2" gate="G$1" pin="1"/>
 <pinref part="U$12" gate="G$1" pin="GND"/>
 </segment>
@@
 <segment>
 <pinref part="U$3" gate="G$1" pin="3.3V"/>
-<pinref part="J3" gate="G$1" pin="2"/>
+<pinref part="J2" gate="G$1" pin="2"/>
 </segment>
 </net>
@@
 <label x="-48.26" y="45.72" size="1.778" layer="95"/>
 <pinref part="U1" gate="G$1" pin="PA31/SWDIO"/>
-<pinref part="J3" gate="G$1" pin="3"/>
+<pinref part="J2" gate="G$1" pin="3"/>
 <wire x1="-40.64" y1="45.72" x2="-60.96" y2="45.72" width="0.1524" layer="91"/>
 </segment>
@@
 <label x="-48.26" y="48.26" size="1.778" layer="95"/>
 <wire x1="-50.8" y1="48.26" x2="-48.26" y2="48.26" width="0.1524" layer="91"/>
-<pinref part="J3" gate="G$1" pin="4"/>
+<pinref part="J2" gate="G$1" pin="4"/>
 <wire x1="-48.26" y1="48.26" x2="-40.64" y2="48.26" width="0.1524" layer="91"/>
 <wire x1="-50.8" y1="48.26" x2="-60.96" y2="48.26" width="0.1524" layer="91"/>
@@
 <segment>
 <pinref part="U1" gate="G$1" pin="PA14/AIN6"/>
-<pinref part="J2" gate="G$1" pin="1"/>
+<pinref part="J3" gate="G$1" pin="1"/>
 <wire x1="-60.96" y1="60.96" x2="-40.64" y2="60.96" width="0.1524" layer="91"/>
 </segment>
@@
 <segment>
 <pinref part="U1" gate="G$1" pin="PA09"/>
-<pinref part="J2" gate="G$1" pin="2"/>
+<pinref part="J3" gate="G$1" pin="2"/>
 <wire x1="-60.96" y1="63.5" x2="-40.64" y2="63.5" width="0.1524" layer="91"/>
 </segment>
@@
 <segment>
 <pinref part="U1" gate="G$1" pin="PA08"/>
-<pinref part="J2" gate="G$1" pin="3"/>
+<pinref part="J3" gate="G$1" pin="3"/>
 <wire x1="-60.96" y1="66.04" x2="-40.64" y2="66.04" width="0.1524" layer="91"/>
 </segment>
@@
 <segment>
 <pinref part="U1" gate="G$1" pin="PA05/AIN3"/>
-<pinref part="J2" gate="G$1" pin="4"/>
+<pinref part="J3" gate="G$1" pin="4"/>
 <wire x1="-60.96" y1="68.58" x2="-40.64" y2="68.58" width="0.1524" layer="91"/>
 </segment>
@@
 <segment>
 <pinref part="U1" gate="G$1" pin="PA28/!RST"/>
-<pinref part="J3" gate="G$1" pin="5"/>
+<pinref part="J2" gate="G$1" pin="5"/>
 <wire x1="-40.64" y1="50.8" x2="-60.96" y2="50.8" width="0.1524" layer="91"/>
 <label x="-48.26" y="50.8" size="1.778" layer="95"/>

Commit message: added values
Parts:
- C5: value 1uF -> 10uF
- C6: value (none) -> 10uF
Changed lines of the file:
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@@
 <part name="FRAME1" library="frames" library_urn="urn:adsk.eagle:library:229" deviceset="A4L-LOC" device=""/>
 <part name="L1" library="microbuilder" deviceset="INDUCTOR" device="TDK_VLC6045"/>
-<part name="C6" library="microbuilder" deviceset="CAP_CERAMIC" device="0603"/>
+<part name="C6" library="microbuilder" deviceset="CAP_CERAMIC" device="0603" value="10uF"/>
 <part name="U$1" library="microbuilder" deviceset="GND" device=""/>
 <part name="U$7" library="microbuilder" deviceset="GND" device=""/>
@@
 <part name="U$8" library="microbuilder" deviceset="GND" device=""/>
 <part name="C4" library="microbuilder" deviceset="CAP_CERAMIC" device="0805" value="10uF"/>
-<part name="C5" library="microbuilder" deviceset="CAP_CERAMIC" device="0603" value="1uF"/>
+<part name="C5" library="microbuilder" deviceset="CAP_CERAMIC" device="0603" value="10uF"/>
 <part name="U$9" library="microbuilder" deviceset="GND" device=""/>
 <part name="U$10" library="microbuilder" deviceset="GND" device=""/>
@@
 </instance>
 <instance part="U3" gate="G$1" x="78.74" y="-27.94" smashed="yes">
-<attribute name="NAME" x="60.9589" y="-19.31945" size="2.08293125" layer="95" ratio="10" rot="SR0"/>
+<attribute name="NAME" x="68.5789" y="-19.31945" size="2.08293125" layer="95" ratio="10" rot="SR0"/>
 <attribute name="VALUE" x="60.9344" y="-39.5767" size="2.0858" layer="96" ratio="10" rot="SR0"/>
 </instance>

Commit message: modified c6 to 1uF
Parts:
- C6: value 10uF -> 1uF
Changed lines of the file:
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@@
 <part name="FRAME1" library="frames" library_urn="urn:adsk.eagle:library:229" deviceset="A4L-LOC" device=""/>
 <part name="L1" library="microbuilder" deviceset="INDUCTOR" device="TDK_VLC6045"/>
-<part name="C6" library="microbuilder" deviceset="CAP_CERAMIC" device="0603" value="10uF"/>
+<part name="C6" library="microbuilder" deviceset="CAP_CERAMIC" device="0603" value="1uF"/>
 <part name="U$1" library="microbuilder" deviceset="GND" device=""/>
 <part name="U$7" library="microbuilder" deviceset="GND" device=""/>
