File: water-pump.brd (EAGLE design)
At the start: 53 x 79.1 mm, 27 parts, among them U1 LDL1117S12R, U3 ATSAMD11C14A-SSUT

Commit message: minor adjustments to water pump
Parts:
- removed 1UF1: (no value), microbuilder:0603
- removed D2: (no value), Adafruit:CHIPLED_0805
- removed J3: (no value), SparkFun-Connectors:1X02_LONGPADS
- removed J4: (no value), SparkFun-Connectors:1X04
- removed R3, R4: (no value), Adafruit:R0805
- added C6: 10uF, microbuilder:0603
- added D6: (no value), Adafruit:CHIPLED_0805
- added F1: (no value), Adafruit:1812
- added J10: (no value), SparkFun-Connectors:1X02_LONGPADS
- added R6: (no value), Adafruit:R0805
- D3: value (none) -> 3A/40V/500mV; device Adafruit:CHIPLED_0805 -> SparkFun-DiscreteSemi:SMA-DIODE
- J1: device EAGLE-INPUT_OUTPUT_CONNECTORS-rev17a:629105136821 -> SparkFun-Connectors:USB-B-MICRO-SMD
- J2: device SparkFun-Connectors:1X02_LONGPADS -> SparkFun-Connectors:1X05
- moved J2 37.9 mm to (4.00, 62.7), turned to 90 degrees
- moved D3 5.37 mm to (17.1, 55.5), turned to 0 degrees
- moved J1 0.64 mm to (1.97, 55.6), turned to 0 degrees
- renumbered 1UF2 to C4, 1UF3 to C5
Connections:
- net SIGNAL renamed BUS
- removed net 12V: C5.2, D1.C, J2.1, U1.3
- removed net N$4: J1.3, U3.10
- removed net N$5: J1.2, U3.9
- new net 3.3V: C4.2, C6.1, J2.2, R6.2, U1.2, U1.4, U3.12
- new net RESET: J2.5, U3.6
- new net USB+: J1.D+, U3.10
- new net USB-: J1.D-, U3.9
- net GND: now also C6.2, J1.GND, J1.SHIELD1, J1.SHIELD2, J1.SHIELD3, J2.1; no longer 1UF1.2, D3.C, J1.5, J1.SHELL, J1.SHELL1, J1.SHELL2, J1.SHELL3, J4.1
- net N$1: now also J1.VBUS; no longer R3.1
- net N$6: now also D1.A, F1.1; no longer J1.1, J3.2
- net N$7: now also D6.A, R6.1; no longer D2.A, R4.1
- net N$8: now also D6.C; no longer D2.C
- net PUMP: now also J10.2; no longer J2.2
- net SWCLK: now also J2.4; no longer J4.4
- net SWDIO: now also J2.3; no longer J4.3
- net VCC: now also C5.2, D1.C, D3.C, J10.1, U1.3; no longer 1UF1.1, C4.2, J4.2, R3.2, R4.2, U1.2, U1.4, U3.12
- net VCC-RAW: now also F1.2; no longer D1.A, J3.1
Routing:
- net 3.3V: track 0.00 -> 37.2 mm, vias 0 -> 2
- net VCC: track 58.3 -> 28.3 mm
- net 12V: track 15.3 -> 0.00 mm
- net RESET: track 0.00 -> 11.6 mm
- net N$1: track 2.79 -> 12.6 mm, vias 0 -> 2
- net N$4: track 9.28 -> 0.00 mm
- net USB+: track 0.00 -> 8.04 mm
- net N$5: track 7.82 -> 0.00 mm
- net USB-: track 0.00 -> 6.84 mm
- net N$6: track 10.0 -> 16.4 mm
- net VCC-RAW: track 96.1 -> 97.9 mm, vias 0 -> 2
- net N$8: track 4.68 -> 6.27 mm
- net PUMP_CTRL: track 40.6 -> 41.9 mm
- net SWDIO: track 10.8 -> 9.89 mm
- net SWCLK: track 8.39 -> 7.58 mm
Other:
- board text added: "BUS"
- board text removed: "LED+"
- board text removed: "Left and Right Side LEDs are mounted different!"
- board text removed: "SIGNAL"
- board text removed: "Sense"

Commit message: modified c6 to 1uF
Parts:
- C6: value 10uF -> 1uF
Changed lines of the file:
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@@
 <attribute name="VALUE" x="7.283" y="70.625" size="0.762" layer="27" font="vector" ratio="15" rot="R270"/>
 </element>
-<element name="C6" library="microbuilder" package="0603" value="10uF" x="12.371" y="56.836" smashed="yes" rot="R180">
+<element name="C6" library="microbuilder" package="0603" value="1uF" x="12.371" y="56.836" smashed="yes" rot="R180">
 <attribute name="NAME" x="10.593" y="56.963" size="0.762" layer="25" font="vector" ratio="15" rot="R180"/>
 <attribute name="VALUE" x="10.593" y="57.598" size="0.4064" layer="27" font="vector" ratio="10" rot="R180"/>
