File: PCB/Fan-Module.brd (EAGLE design)
At the start: 58 x 66 mm, 28 parts, among them U1 ATSAMD11C14A-SSUT_ATSAMD11C14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, U3 LDL1117S12R_LDL1117S12R

Commit message: added b/tstop and b/restricted to write address on pcb
Parts:
- moved R1 10.9 mm to (57.5, 27.5)
Routing:
- net BUS: track 52.5 -> 63.9 mm
- net N$3: track 45.3 -> 34.6 mm
Changed lines of the file:
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@@
 <drawing>
 <settings>
-<setting alwaysvectorfont="no"/>
+<setting alwaysvectorfont="yes"/>
 <setting keepoldvectorfont="yes"/>
 <setting verticaltext="up"/>
@@
 <text x="23.454" y="5.73" size="1.016" layer="25">VCC</text>
 <text x="21.168" y="16.144" size="1.27" layer="21" font="vector">+</text>
+<polygon width="0.1524" layer="29">
+<vertex x="55.813" y="64.15"/>
+<vertex x="55.813" y="46.07"/>
+<vertex x="63.249" y="46.07"/>
+<vertex x="63.249" y="64.15"/>
+</polygon>
+<polygon width="0.1524" layer="30">
+<vertex x="55.813" y="46.086"/>
+<vertex x="55.813" y="64.166"/>
+<vertex x="63.249" y="64.166"/>
+<vertex x="63.249" y="46.086"/>
+</polygon>
+<polygon width="0.1524" layer="41">
+<vertex x="55.813" y="64.15"/>
+<vertex x="55.813" y="46.07"/>
+<vertex x="63.249" y="46.07"/>
+<vertex x="63.249" y="64.15"/>
+</polygon>
+<polygon width="0.1524" layer="42">
+<vertex x="55.813" y="46.086"/>
+<vertex x="55.813" y="64.166"/>
+<vertex x="63.249" y="64.166"/>
+<vertex x="63.249" y="46.086"/>
+</polygon>
 </plain>
 <attributes>
@@
 <attribute name="VALUE" x="57.785" y="21.717" size="0.6096" layer="27" font="vector" ratio="20" rot="R270"/>
 </element>
-<element name="R1" library="rcl" library_urn="urn:adsk.eagle:library:334" package="R1206" package3d_urn="urn:adsk.eagle:package:23540/2" value="2k" x="57.023" y="38.379" smashed="yes" rot="R270">
-<attribute name="NAME" x="56.896" y="35.839" size="0.8128" layer="25" ratio="18" rot="R270"/>
-<attribute name="SPICEPREFIX" value="R" x="57.023" y="38.379" size="1.778" layer="27" rot="R270" display="off"/>
-<attribute name="VALUE" x="56.388" y="35.839" size="0.4064" layer="27" ratio="10" rot="R270"/>
+<element name="R1" library="rcl" library_urn="urn:adsk.eagle:library:334" package="R1206" package3d_urn="urn:adsk.eagle:package:23540/2" value="2k" x="57.531" y="27.457" smashed="yes" rot="R270">
+<attribute name="NAME" x="57.404" y="24.917" size="0.8128" layer="25" ratio="18" rot="R270"/>
+<attribute name="SPICEPREFIX" value="R" x="57.531" y="27.457" size="1.778" layer="27" rot="R270" display="off"/>
+<attribute name="VALUE" x="56.896" y="24.917" size="0.4064" layer="27" ratio="10" rot="R270"/>
 </element>
 <element name="R6" library="rcl" library_urn="urn:adsk.eagle:library:334" package="R0805" package3d_urn="urn:adsk.eagle:package:23553/2" value="59R" x="44.069" y="6.477" smashed="yes">
@@
 <wire x1="29.591" y1="11.43" x2="28.194" y2="10.033" width="0.4064" layer="1"/>
 <wire x1="28.194" y1="10.033" x2="27.522" y2="10.033" width="0.4064" layer="1"/>
-<wire x1="49.498" y1="66.646" x2="52.15" y2="64" width="0" layer="19" extent="1-1"/>
-<wire x1="46.85" y1="64" x2="49.498" y2="66.646" width="0" layer="19" extent="1-1"/>
-<wire x1="49.498" y1="61.346" x2="52.15" y2="64" width="0" layer="19" extent="1-1"/>
-<wire x1="12.888" y1="45.482" x2="46.85" y2="64" width="0" layer="19" extent="1-1"/>
-<wire x1="8.128" y1="44.933" x2="12.888" y2="45.146" width="0" layer="19" extent="1-1"/>
-<wire x1="8.001" y1="27.053" x2="8.128" y2="44.933" width="0" layer="19" extent="1-1"/>
-<wire x1="8.001" y1="23.368" x2="8.001" y2="27.053" width="0" layer="19" extent="1-1"/>
-<wire x1="10.726" y1="22.068" x2="8.001" y2="23.368" width="0" layer="19" extent="1-1"/>
-<wire x1="8.001" y1="19.683" x2="10.726" y2="22.068" width="0" layer="19" extent="1-1"/>
-<wire x1="12.28" y1="18.288" x2="10.726" y2="22.068" width="0" layer="19" extent="1-1"/>
-<wire x1="12.714" y1="15.85" x2="12.28" y2="18.288" width="0" layer="19" extent="1-1"/>
-<wire x1="24.511" y1="7.962" x2="27.522" y2="10.033" width="0" layer="19" extent="1-1"/>
-<wire x1="17.653" y1="7.708" x2="17.272" y2="14.40815" width="0" layer="19" extent="1-16"/>
-<wire x1="46.85" y1="10.5" x2="29.591" y2="11.43" width="0" layer="19" extent="1-1"/>
-<wire x1="49.498" y1="13.146" x2="46.85" y2="10.5" width="0" layer="19" extent="1-1"/>
-<wire x1="52.15" y1="10.5" x2="49.498" y2="13.146" width="0" layer="19" extent="1-1"/>
-<wire x1="49.498" y1="7.846" x2="46.85" y2="10.5" width="0" layer="19" extent="1-1"/>
-<wire x1="59.817" y1="20.447" x2="52.15" y2="10.5" width="0" layer="19" extent="1-1"/>
 </signal>
 <signal name="VCC-RAW" class="1">
@@
 <wire x1="36.15" y1="64" x2="33.498" y2="61.348" width="0.6096" layer="1"/>
 <wire x1="33.498" y1="61.348" x2="33.498" y2="61.346" width="0.6096" layer="1"/>
-<wire x1="57.023" y1="39.801" x2="57.023" y2="51.181" width="0.4064" layer="1"/>
-<wire x1="57.023" y1="51.181" x2="51.308" y2="56.896" width="0.4064" layer="1"/>
-<wire x1="51.308" y1="56.896" x2="43.252" y2="56.896" width="0.4064" layer="1"/>
+<wire x1="54.737" y1="53.848" x2="54.737" y2="31.673" width="0.4064" layer="1"/>
+<wire x1="57.531" y1="28.879" x2="54.737" y2="31.673" width="0.4064" layer="1"/>
+<wire x1="54.737" y1="53.848" x2="51.689" y2="56.896" width="0.4064" layer="1"/>
+<wire x1="51.689" y1="56.896" x2="43.252" y2="56.896" width="0.4064" layer="1"/>
 <wire x1="43.252" y1="56.896" x2="36.15" y2="63.998" width="0.4064" layer="1"/>
 </signal>
@@
 <wire x1="42.672" y1="11.303" x2="47.752" y2="16.383" width="0.4064" layer="1"/>
 <wire x1="47.752" y1="16.383" x2="53.721" y2="16.383" width="0.4064" layer="1"/>
-<wire x1="53.721" y1="16.383" x2="57.023" y2="19.685" width="0.4064" layer="1"/>
-<wire x1="57.023" y1="19.685" x2="57.023" y2="36.957" width="0.4064" layer="1"/>
+<wire x1="53.721" y1="16.383" x2="57.531" y2="20.193" width="0.4064" layer="1"/>
+<wire x1="57.531" y1="20.193" x2="57.531" y2="26.035" width="0.4064" layer="1"/>
 </signal>
 <signal name="N$8">
